File: cad/harmonic_jerkulator.kicad_pcb (KiCad board)
At the start: 2 copper layers, 91 x 87 mm, 45 parts, among them J101 JACK_IN, J102 JACK_OUT, J103 CONN_PSU, J105 PNP, J106 NPN, J107 SW_BYPASS, J108 DIODE1, J109 DIODE_SW, J110 DIODE2, J111 Conn_01x06, J113 Conn_01x06, K101 TQ2SA-5V, Q101 BC850, Q102 BC856, Q103 DTC123Y, Q104 DTC123Y, Q105 DTA114E, U101 4013

Commit message: Corrected PCB revision number.
Other:
- board text added: "RANDAGODRON harmonic jerkulator v03"
- board text added: "jerkulator v03"
- board text removed: "RANDAGODRON harmonic jerkulator v02"
- board text removed: "jerkulator v02"
Changed lines of the file:
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@@
   (gr_line (start 74.8 83.5) (end 158 83.5) (layer Eco2.User) (width 0.2))
   (gr_line (start 74.8 78) (end 158 78) (layer Eco2.User) (width 0.2))
-  (gr_text "jerkulator v02" (at 91 103) (layer B.Cu)
+  (gr_text "jerkulator v03" (at 91 103) (layer B.Cu)
     (effects (font (size 1 1) (thickness 0.2)) (justify mirror))
   )
@@
     (effects (font (size 1 1) (thickness 0.2)) (justify left mirror))
   )
-  (gr_text "RANDAGODRON\nharmonic \njerkulator v02" (at 152.75 106.75) (layer B.Cu)
+  (gr_text "RANDAGODRON\nharmonic \njerkulator v03" (at 152.75 106.75) (layer B.Cu)
     (effects (font (size 1 1) (thickness 0.25)) (justify left mirror))
   )
@@
   (target plus (at 67.2 129.6) (size 5) (width 0.15) (layer Edge.Cuts))
   (target plus (at 93.6 49.2) (size 5) (width 0.15) (layer Edge.Cuts))
-  (gr_text "jerkulator v02" (at 91 103) (layer F.Cu)
+  (gr_text "jerkulator v03" (at 91 103) (layer F.Cu)
     (effects (font (size 1 1) (thickness 0.2)))
   )
@@
     (effects (font (size 1 1) (thickness 0.2)) (justify left))
   )
-  (gr_text "RANDAGODRON\nharmonic \njerkulator v02" (at 142.05 106.7) (layer F.Cu)
+  (gr_text "RANDAGODRON\nharmonic \njerkulator v03" (at 142.05 106.7) (layer F.Cu)
     (effects (font (size 1 1) (thickness 0.25)) (justify left))
   )
